File: hardware/electronics/electronics/electronics.kicad_sch (KiCad schematic)
At the start: 15 parts, among them J1 Conn_Coaxial_Small, M1 Parachute_Servo, M2 Parachute_Servo, Q1 BC547, SW1 RBF, U1 RFM95W-915S2, U2 BMP585, U3 LSM6DS3, U4 SD Card mini module, U5 ESP32-S3-DEVKITC-1-N8R2, U6 GPS M8N, U7 MINI 560 STEP DOWN

Commit message: fix: hardware kicad schematic resistor correction
R1 (servo signal) 1k->220Ω per bench measurement. The 1k pull-up on
the servo PWM line was clamping the ESP32-S3 GPIO39 output swing,
causing intermittent servo position jitter in the bench test.

This is the hardware root cause that compounded the SERVO_PIN=7->39
pin mapping fix: even with the correct pin, the wrong resistor value
would prevent clean servo actuation.

Only the .kicad_sch is committed — the .kicad_prl is a KiCad GUI
session artifact and is not meaningful to track.
Parts:
- R1: value 1k -> 220
Changed lines of the file:
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@@
 			)
 		)
-		(property "Value" "1k"
+		(property "Value" "220"
 			(at 116.84 138.43 90)
 			(show_name no)
